File: Schematics/Epiphone Blues Custom 30.kicad_sch (KiCad schematic)
At the start: 274 parts, among them J3 Conn_Coaxial_Power, M1 Fan, SW2 EQ mode, SW3 POWER, SW4 STANDBY, SW5 PENTODE

Commit message: Updated output
Parts:
- C1: value 22uF/50V -> 22µF/50V
- C15, C21, C22, C8: value 22uF/35V -> 22µF/35V
- C24: value 47p/2KV -> 47pF/2KV
- C28: value 0.1uF/400V -> 0.1µF/400V
- C29: value 100uF/100V -> 100µF/100V
- C3: value 22000uF/25V -> 22000µF/25V
- C30, C31: value 22uF/450V -> 22µF/450V
- C32: value 47uF/450V -> 47µF/450V
- C33, C34, C35: value 100uF/400V -> 100µF/400V
- C36: value C_Polarized -> 100µF/400V
Connections:
- net at FCR.: now also B., C33.1, R49.1; no longer TRF4.
- net at SS1.: now also F4.1; no longer SW4.
- net at 0VAC.: now also TR2.; no longer PT3.
- net at 60VAC.: now also TR2.; no longer PT11.
- net at PT2.: now also PT3., PT6. (x2)
- net at V7.: now also C29.1, R44.2, V6.
- net at PT5.: now also PT6. (x2)
- net at PT6.: no longer PT5. (x2)
- net at PT4.: now also PT1., PT7.
- net at ff.: now also BLUE.; no longer TR3.
- net at BLUE.: now also OT6.; no longer ff.
- net at PT7.: now also PT1.
- net at PT1.: no longer PT7.
- net at U?.: now also OUT1.; no longer TR3.
- net at OUT1.: now also PS1., V6.; no longer U?.
- net at 120VAC.: now also TR2.; no longer PT5.
- net at TR3.: now also d.; no longer d.
- net at a.: now also d.; no longer TR3.
- net at s.: now also d.; no longer TR3.
- net at d.: now also s.; no longer TR3.
- net at PT7.: now also 100VAC.
- net at 100VAC.: now also TR2.; no longer PT7.
- net at 5VAC.: now also PT13.
- net at PT13.: now also C35.1, HTFS., R50.1, V8.; no longer 5VAC.
- net at BLK.: now also SW3.; no longer PT1.
- net at SW3.: now also BLU.; no longer BLK.
- net at 0VAC.: now also TR2.; no longer PT6.
- net at 100VAC.: now also TR2.; no longer PT4.
- net at V6., V7.: now also PT15.; no longer PT14.
- net at PT1.: now also PT8.
- net at PT8.: no longer PT1.
- net at SW2.: now also RV7.; no longer RV5.
- net at RV7.: now also R23.2; no longer SW2.
- net at 120VAC.: now also TR2.; no longer PT8.
- net at SW4.: now also 350VAC.; no longer 350VAC.
- net at 350VAC.: now also TR2.; no longer SW4.
- net at PT2.: now also PT3.
- net at PT3.: no longer PT2.
- net at PT5.: now also PT1., PT8.
- net at 0VAC.: now also PT12.
- net at PT12.: now also F7.1; no longer 0VAC.
- net at s.: now also a.; no longer d.
- net at a.: now also J6., J7.; no longer s.
- net at BRN.: now also F9.2; no longer SW3.
- net at BLU.: now also AC-Input1.; no longer SW3.
- net at PT3.: now also PT2.
- net at PT2.: no longer PT3.
- new net: C3.1, D6.1 (K), D7.1 (K), F., M1. (-), V1., V2., V3., V4., V5.
- new net: FCR., TRF4.
- new net: SS1., SW4.
- new net: 0VAC., PT3.
- new net: 0VAC., TR2. (x2)
- new net: D4.2 (A), J4., RL3.
- new net: D3.2 (A), J4., RL1., RLY2.
- new net: J4., PB1.
- new net: 60VAC., PT11.
- new net: J3. (In), R29.1, RL3., V5A., V5B.
- new net: OUT2., PS2., V7.
- new net: TR3., ff.
- new net: TR3., U?.
- new net: B., PS5., PS6.
- new net: J5., J6., J7., J8., J9., d.
- new net: C4.2, RLY2., RV1.
- new net: 120VAC., PT5.
- new net: R19.2, RLY2., V2B.
- new net: RLY2., RV4.
- new net: TR3., d.
- new net: TR3., a.
- new net: TR3., s.
- new net: BLK., PT1.
- new net: 0VAC., PT6.
- new net: 100VAC., PT4.
- new net: PT14., V6., V7.
- new net: C17.2, RV7., SW2.
- new net: RV5., SW2.
- new net: 120VAC., PT8.
- new net: 350VAC., SW4.
- new net: C6.2, RL1., RV2., V1B.
- new net: BRN., SW3.
- new net: J2. (In), T1. (SB)
- now unconnected: PT1., PT1., PT3., PT3., PT6., PT6., PT7., PT8., V6., V6.
Other:
- title: Epiphone Blues Custom 30 -> Epiphone Blues Custom 30 : Version-2006-060622-DPPT
Changed lines of the file:
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@@
 	(paper "A3")
 	(title_block
-		(title "Epiphone Blues Custom 30")
-		(date "2024/11/02")
+		(title "Epiphone Blues Custom 30 : Version-2006-060622-DPPT")
+		(date "2024/11/07")
 		(rev "1")
 		(comment 1 "Creator : Geert Peeters")
@@
 	(wire
 		(pts
-			(xy 251.206 243.84) (xy 251.46 243.84)
-		)
-		(stroke
-			(width 0)
-			(type default)
-			(color 0 0 255 1)
-		)
-	)
-	(wire
-		(pts
 			(xy 290.068 158.242) (xy 295.656 158.242)
 		)
@@
 	(wire
 		(pts
-			(xy 251.46 243.84) (xy 251.46 245.11)
+			(xy 251.206 243.84) (xy 251.206 245.11)
 		)
 		(stroke
@@
 			)
 		)
-		(property "Value" "22uF/450V"
+		(property "Value" "22µF/450V"
 			(at 354.076 226.568 0)
 			(effects
@@
 			)
 		)
-		(property "Value" "22uF/35V"
+		(property "Value" "22µF/35V"
 			(at 138.176 64.262 0)
 			(effects
@@
 		)
 		(property "Value" "220K/2W"
-			(at 242.824 225.806 90)
+			(at 243.078 226.314 90)
 			(effects
 				(font
@@
 			)
 		)
-		(property "Value" "47uF/450V"
+		(property "Value" "47µF/450V"
 			(at 339.8025 226.5221 0)
 			(effects
@@
 			)
 		)
-		(property "Value" "22uF/35V"
+		(property "Value" "22µF/35V"
 			(at 224.282 141.986 0)
 			(effects
@@
 			)
 		)
-		(property "Value" "22uF/35V"
+		(property "Value" "22µF/35V"
 			(at 146.558 145.034 0)
 			(effects
@@
 			)
 		)
-		(property "Value" "22uF/450V"
+		(property "Value" "22µF/450V"
 			(at 368.3 226.822 0)
 			(effects
@@
 			)
 		)
-		(property "Value" "100uF/100V"
+		(property "Value" "100µF/100V"
 			(at 323.7104 183.6435 90)
 			(effects
@@
 			)
 		)
-		(property "Value" "22uF/35V"
+		(property "Value" "22µF/35V"
 			(at 243.84 80.518 0)
 			(effects
@@
 			)
 		)
-		(property "Value" "100uF/400V"
+		(property "Value" "100µF/400V"
 			(at 325.882 236.728 0)
 			(effects
@@
 			)
 		)
-		(property "Value" "22000uF/25V"
+		(property "Value" "22000µF/25V"
 			(at 237.3986 274.0401 0)
 			(effects
@@
 			)
 		)
-		(property "Value" "100uF/400V"
+		(property "Value" "100µF/400V"
 			(at 325.882 226.568 0)
 			(effects
@@
 		(dnp no)
 		(property "Reference" "C35"
-			(at 254.254 220.472 0)
+			(at 254 221.488 0)
 			(effects
 				(font
@@
 			)
 		)
-		(property "Value" "100uF/400V"
-			(at 254.508 222.504 0)
+		(property "Value" "100µF/400V"
+			(at 254 223.012 0)
 			(effects
 				(font
@@
 			)
 		)
-		(property "Value" "47p/2KV"
+		(property "Value" "47pF/2KV"
 			(at 313.4604 55.7963 90)
 			(effects
@@
 			)
 		)
-		(property "Value" "0.1uF/400V"
+		(property "Value" "0.1µF/400V"
 			(at 318.262 94.996 0)
 			(effects
@@
 		(dnp no)
 		(property "Reference" "C36"
-			(at 253.746 235.712 0)
+			(at 253.746 235.966 0)
 			(effects
 				(font
@@
 			)
 		)
-		(property "Value" "C_Polarized"
-			(at 255.27 237.363 0)
+		(property "Value" "100µF/400V"
+			(at 253.746 237.49 0)
 			(effects
 				(font
@@
 	(symbol
 		(lib_id "power:GND")
-		(at 251.46 245.11 0)
+		(at 251.206 245.11 0)
 		(unit 1)
 		(exclude_from_sim no)
@@
 		(fields_autoplaced yes)
 		(property "Reference" "#PWR03"
-			(at 251.46 251.46 0)
+			(at 251.206 251.46 0)
 			(effects
 				(font
@@
 		)
 		(property "Value" "GND"
-			(at 251.46 250.19 0)
+			(at 251.206 250.19 0)
 			(effects
 				(font
@@
 		)
 		(property "Footprint" ""
-			(at 251.46 245.11 0)
+			(at 251.206 245.11 0)
 			(effects
 				(font
@@
 		)
 		(property "Datasheet" ""
-			(at 251.46 245.11 0)
+			(at 251.206 245.11 0)
 			(effects
 				(font
@@
 		)
 		(property "Description" "Power symbol creates a global label with name \"GND\" , ground"
-			(at 251.46 245.11 0)
+			(at 251.206 245.11 0)
 			(effects
 				(font
@@
 			)
 		)
-		(property "Value" "22uF/50V"
+		(property "Value" "22µF/50V"
 			(at 74.93 73.66 0)
 			(effects
