File: Schematics/Epiphone Blues Custom 30.kicad_sch (KiCad schematic)
At the start: 274 parts, among them J3 Conn_Coaxial_Power, M1 Fan, SW2 EQ mode, SW3 POWER, SW4 STANDBY, SW5 PENTODE

Commit message: pulled symbol library from version 2005 mods
Parts:
- C3: value 22000uF/25V -> 471/1KV
Connections:
- net GND: no longer C3.2
- net at FCR.: now also B., C33.1, R49.1; no longer TRF4.
- net at C2.2, C5.1, R5.1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: no longer C3.1
- net at SS1.: now also F4.1; no longer SW4.
- net at 0VAC.: now also TR2.; no longer PT3.
- net at 60VAC.: now also TR2.; no longer PT11.
- net at PT2.: now also PT3., PT6. (x2)
- net at V7.: now also C29.1, R44.2, V6.
- net at PT5.: now also PT6. (x2)
- net at PT6.: no longer PT5. (x2)
- net at PT4.: now also PT1., PT7.
- net at ff.: now also BLUE.; no longer TR3.
- net at BLUE.: now also OT6.; no longer ff.
- net at PT7.: now also PT1.
- net at PT1.: no longer PT7.
- net at U?.: now also OUT1.; no longer TR3.
- net at OUT1.: now also PS1., V6.; no longer U?.
- net at 120VAC.: now also TR2.; no longer PT5.
- net at TR3.: now also d.; no longer d.
- net at a.: now also d.; no longer TR3.
- net at s.: now also d.; no longer TR3.
- net at d.: now also s.; no longer TR3.
- net at PT7.: now also 100VAC.
- net at 100VAC.: now also TR2.; no longer PT7.
- net at 5VAC.: now also PT13.
- net at PT13.: now also C35.1, HTFS., R50.1, V8.; no longer 5VAC.
- net at BLK.: now also SW3.; no longer PT1.
- net at SW3.: now also BLU.; no longer BLK.
- net at 0VAC.: now also TR2.; no longer PT6.
- net at 100VAC.: now also TR2.; no longer PT4.
- net at V6., V7.: now also PT15.; no longer PT14.
- net at PT1.: now also PT8.
- net at PT8.: no longer PT1.
- net at SW2.: now also RV7.; no longer RV5.
- net at RV7.: now also R23.2; no longer SW2.
- net at 120VAC.: now also TR2.; no longer PT8.
- net at SW4.: now also 350VAC.; no longer 350VAC.
- net at 350VAC.: now also TR2.; no longer SW4.
- net at PT2.: now also PT3.
- net at PT3.: no longer PT2.
- net at PT5.: now also PT1., PT8.
- net at 0VAC.: now also PT12.
- net at PT12.: now also F7.1; no longer 0VAC.
- net at s.: now also a.; no longer d.
- net at a.: now also J6., J7.; no longer s.
- net at BRN.: now also F9.2; no longer SW3.
- net at BLU.: now also AC-Input1.; no longer SW3.
- net at PT3.: now also PT2.
- net at PT2.: no longer PT3.
- new net: D6.1 (K), D7.1 (K), F., M1. (-), V1., V2., V3., V4., V5.
- new net: FCR., TRF4.
- new net: SS1., SW4.
- new net: 0VAC., PT3.
- new net: 0VAC., TR2. (x2)
- new net: D4.2 (A), J4., RL3.
- new net: D3.2 (A), J4., RL1., RLY2.
- new net: J4., PB1.
- new net: 60VAC., PT11.
- new net: J3. (In), R29.1, RL3., V5A., V5B.
- new net: OUT2., PS2., V7.
- new net: TR3., ff.
- new net: TR3., U?.
- new net: B., PS5., PS6.
- new net: J5., J6., J7., J8., J9., d.
- new net: C4.2, RLY2., RV1.
- new net: 120VAC., PT5.
- new net: R19.2, RLY2., V2B.
- new net: RLY2., RV4.
- new net: TR3., d.
- new net: TR3., a.
- new net: TR3., s.
- new net: BLK., PT1.
- new net: 0VAC., PT6.
- new net: 100VAC., PT4.
- new net: PT14., V6., V7.
- new net: C17.2, RV7., SW2.
- new net: RV5., SW2.
- new net: 120VAC., PT8.
- new net: 350VAC., SW4.
- new net: C6.2, RL1., RV2., V1B.
- new net: BRN., SW3.
- new net: J2. (In), T1. (SB)
- now unconnected: C3.1, PT1., PT1., PT3., PT3., PT6., PT6., PT7., PT8., V6., V6.
Other:
- moved on the sheet: C3
Changed lines of the file:
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@@
 	)
 	(junction
-		(at 108.712 64.77)
-		(diameter 0)
-		(color 194 0 0 1)
-	)
-	(junction
 		(at 149.352 54.61)
 		(diameter 0)
@@
 	)
 	(junction
+		(at 108.712 64.77)
+		(diameter 0)
+		(color 0 0 0 0)
+	)
+	(junction
 		(at 241.046 36.322)
 		(diameter 0)
@@
 	(wire
 		(pts
+			(xy 108.712 50.546) (xy 108.712 52.324)
+		)
+		(stroke
+			(width 0)
+			(type default)
+			(color 0 0 255 1)
+		)
+	)
+	(wire
+		(pts
 			(xy 308.356 25.908) (xy 308.356 22.098)
 		)
@@
 	(wire
 		(pts
-			(xy 108.712 61.722) (xy 108.712 64.77)
-		)
-		(stroke
-			(width 0)
-			(type default)
-			(color 0 0 255 1)
-		)
-	)
-	(wire
-		(pts
 			(xy 324.358 73.152) (xy 314.452 73.152)
 		)
@@
 	(wire
 		(pts
+			(xy 108.712 63.246) (xy 108.712 64.77)
+		)
+		(stroke
+			(width 0)
+			(type default)
+		)
+	)
+	(wire
+		(pts
 			(xy 249.174 280.67) (xy 255.27 280.67)
 		)
@@
 	(wire
 		(pts
-			(xy 108.712 54.102) (xy 108.712 50.546)
-		)
-		(stroke
-			(width 0)
-			(type default)
-			(color 0 0 255 1)
-		)
-	)
-	(wire
-		(pts
 			(xy 275.336 178.816) (xy 278.892 178.816)
 		)
@@
 	)
 	(symbol
+		(lib_name "C_1")
 		(lib_id "Device:C")
-		(at 108.712 57.912 0)
+		(at 108.712 61.214 0)
 		(unit 1)
 		(exclude_from_sim no)
@@
 		(dnp no)
 		(property "Reference" "C3"
-			(at 111.252 57.912 0)
+			(at 111.252 61.214 0)
 			(effects
 				(font
@@
 		)
 		(property "Value" "471/1KV"
-			(at 108.966 59.944 0)
+			(at 108.966 63.246 0)
 			(effects
 				(font
@@
 		)
 		(property "Footprint" ""
-			(at 109.6772 61.722 0)
+			(at 109.6772 65.024 0)
 			(effects
 				(font
@@
 		)
 		(property "Datasheet" "~"
-			(at 108.712 57.912 0)
+			(at 108.712 61.214 0)
 			(effects
 				(font
@@
 		)
 		(property "Description" "Unpolarized capacitor"
-			(at 108.712 57.912 0)
+			(at 108.712 61.214 0)
 			(effects
 				(font
@@
 	)
 	(symbol
+		(lib_name "C_Polarized_1")
 		(lib_id "Device:C_Polarized")
 		(at 234.95 273.304 0)
@@
 		(dnp no)
 		(property "Reference" "C3"
-			(at 236.1286 270.9921 0)
+			(at 237.49 273.304 0)
 			(effects
 				(font
@@
 			)
 		)
-		(property "Value" "22000uF/25V"
-			(at 237.3986 274.0401 0)
+		(property "Value" "471/1KV"
+			(at 235.204 275.336 0)
 			(effects
 				(font
@@
 			)
 		)
-		(property "Description" "Polarized capacitor"
+		(property "Description" "Unpolarized capacitor"
 			(at 234.95 273.304 0)
 			(effects

Commit message: add modifications partially
Parts:
- removed SW4: STANDBY, symbol Epi-BC-30:2PST
- added R52, R53: 68R/25W, symbol Device:R
- added SW1, SW6, SW7: ~, symbol Epi-BC-30:SPST-Small
Connections:
- net at FCR.: now also B., C33.1, R49.1; no longer TRF4.
- net at C2.2, C5.1, R5.1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: now also SW1.
- net at SS1.: now also F4.1
- net at 0VAC.: now also TR2.; no longer PT3.
- net at 60VAC.: now also TR2.; no longer PT11.
- net at PT2.: now also PT3., PT6. (x2)
- net at V7.: now also C29.1, R44.2, V6.
- net at PT5.: now also PT6. (x2)
- net at PT6.: no longer PT5. (x2)
- net at C6.1, R6.2, RV2.: now also SW6.; no longer C5.2
- net at PT4.: now also PT1., PT7.
- net at ff.: now also BLUE.; no longer TR3.
- net at BLUE.: now also OT6.; no longer ff.
- net at PT7.: now also PT1.
- net at PT1.: no longer PT7.
- net at U?.: now also OUT1.; no longer TR3.
- net at OUT1.: now also PS1., V6.; no longer U?.
- net at 120VAC.: now also TR2.; no longer PT5.
- net at TR3.: now also d.; no longer d.
- net at a.: now also d.; no longer TR3.
- net at s.: now also d.; no longer TR3.
- net at d.: now also s.; no longer TR3.
- net at PT7.: now also 100VAC.
- net at 100VAC.: now also TR2.; no longer PT7.
- net at 5VAC.: now also PT13.
- net at PT13.: now also C35.1, HTFS., R50.1, V8.; no longer 5VAC.
- net at BLK.: now also SW3.; no longer PT1.
- net at SW3.: now also BLU.; no longer BLK.
- net at 0VAC.: now also TR2.; no longer PT6.
- net at 100VAC.: now also TR2.; no longer PT4.
- net at V6., V7.: now also PT15.; no longer PT14.
- net at PT1.: now also PT8.
- net at PT8.: no longer PT1.
- net at SW2.: now also RV7.; no longer RV5.
- net at RV7.: now also R23.2; no longer SW2.
- net at 120VAC.: now also TR2.; no longer PT8.
- net at SS2.: now also R52.2
- net at 350VAC.: now also TR2. (x2)
- net at PT2.: now also PT3.
- net at PT3.: no longer PT2.
- net at C3.1: now also SW1.
- net at PT5.: now also PT1., PT8.
- net at 0VAC.: now also PT12.
- net at PT12.: now also F7.1; no longer 0VAC.
- net at s.: now also a.; no longer d.
- net at a.: now also J6., J7.; no longer s.
- net at BRN.: now also F9.2; no longer SW3.
- net at BLU.: now also AC-Input1.; no longer SW3.
- net at PT3.: now also PT2.
- net at PT2.: no longer PT3.
- net at C9.2, R9.2: now also SW7.; no longer C10.1
- new net: D6.1 (K), D7.1 (K), F., M1. (-), V1., V2., V3., V4., V5.
- new net: FCR., TRF4.
- new net: R53.2, SS1.
- new net: 0VAC., PT3.
- new net: 0VAC., TR2. (x2)
- new net: D4.2 (A), J4., RL3.
- new net: D3.2 (A), J4., RL1., RLY2.
- new net: J4., PB1.
- new net: 60VAC., PT11.
- new net: J3. (In), R29.1, RL3., V5A., V5B.
- new net: OUT2., PS2., V7.
- new net: C5.2, SW6.
- new net: TR3., ff.
- new net: TR3., U?.
- new net: B., PS5., PS6.
- new net: J5., J6., J7., J8., J9., d.
- new net: C4.2, RLY2., RV1.
- new net: 120VAC., PT5.
- new net: R19.2, RLY2., V2B.
- new net: RLY2., RV4.
- new net: C10.1, SW7.
- new net: TR3., d.
- new net: TR3., a.
- new net: TR3., s.
- new net: BLK., PT1.
- new net: 0VAC., PT6.
- new net: 100VAC., PT4.
- new net: PT14., V6., V7.
- new net: C17.2, RV7., SW2.
- new net: RV5., SW2.
- new net: 120VAC., PT8.
- new net: 350VAC., R53.1
- new net: C6.2, RL1., RV2., V1B.
- new net: 350VAC., R52.1
- new net: BRN., SW3.
- new net: J2. (In), T1. (SB)
- now unconnected: PT1., PT1., PT3., PT3., PT6., PT6., PT7., PT8., V6., V6.
Other:
- moved on the sheet: C10, C5

Commit message: Actual modifications version 2006
Parts:
- added R15': 1K/1W, symbol Device:R
- added R21': 2K7/1W, symbol Device:R
- R15: value 2K2/1W -> 10K/1W
- R21: value 2K2/1W -> 1K5/1W
Connections:
- net GND: now also R15'.2, R21'.1
- net at FCR.: now also B., C33.1, R49.1; no longer TRF4.
- net at 0VAC.: now also TR2.; no longer PT3.
- net at 60VAC.: now also TR2.; no longer PT11.
- net at PT2.: now also PT3., PT6. (x2)
- net at V7.: now also C29.1, R44.2, V6.
- net at PT5.: now also PT6. (x2)
- net at PT6.: no longer PT5. (x2)
- net at PT4.: now also PT1., PT7.
- net at ff.: now also BLUE.; no longer TR3.
- net at BLUE.: now also OT6.; no longer ff.
- net at PT7.: now also PT1.
- net at PT1.: no longer PT7.
- net at U?.: now also OUT1.; no longer TR3.
- net at OUT1.: now also PS1., V6.; no longer U?.
- net at 120VAC.: now also TR2.; no longer PT5.
- net at TR3.: now also d.; no longer d.
- net at a.: now also d.; no longer TR3.
- net at s.: now also d.; no longer TR3.
- net at d.: now also s.; no longer TR3.
- net at PT7.: now also 100VAC.
- net at 100VAC.: now also TR2.; no longer PT7.
- net at 5VAC.: now also PT13.
- net at PT13.: now also C35.1, HTFS., R50.1, V8.; no longer 5VAC.
- net at BLK.: now also SW3.; no longer PT1.
- net at SW3.: now also BLU.; no longer BLK.
- net at R15.1, V2A.: now also R15'.1
- net at 0VAC.: now also TR2.; no longer PT6.
- net at 100VAC.: now also TR2.; no longer PT4.
- net at V6., V7.: now also PT15.; no longer PT14.
- net at PT1.: now also PT8.
- net at PT8.: no longer PT1.
- net at SW2.: now also RV7.; no longer RV5.
- net at RV7.: now also R23.2; no longer SW2.
- net at 120VAC.: now also TR2.; no longer PT8.
- net at PT2.: now also PT3.
- net at PT3.: no longer PT2.
- net at PT5.: now also PT1., PT8.
- net at 0VAC.: now also PT12.
- net at PT12.: now also F7.1; no longer 0VAC.
- net at s.: now also a.; no longer d.
- net at a.: now also J6., J7.; no longer s.
- net at C15.1, R21.2, V2B.: now also R21'.2
- net at BRN.: now also F9.2; no longer SW3.
- net at BLU.: now also AC-Input1.; no longer SW3.
- net at PT3.: now also PT2.
- net at PT2.: no longer PT3.
- new net: D6.1 (K), D7.1 (K), F., M1. (-), V1., V2., V3., V4., V5.
- new net: FCR., TRF4.
- new net: 0VAC., PT3.
- new net: 0VAC., TR2. (x2)
- new net: D4.2 (A), J4., RL3.
- new net: D3.2 (A), J4., RL1., RLY2.
- new net: J4., PB1.
- new net: 60VAC., PT11.
- new net: J3. (In), R29.1, RL3., V5A., V5B.
- new net: OUT2., PS2., V7.
- new net: TR3., ff.
- new net: TR3., U?.
- new net: B., PS5., PS6.
- new net: J5., J6., J7., J8., J9., d.
- new net: C4.2, RLY2., RV1.
- new net: 120VAC., PT5.
- new net: R19.2, RLY2., V2B.
- new net: RLY2., RV4.
- new net: TR3., d.
- new net: TR3., a.
- new net: TR3., s.
- new net: BLK., PT1.
- new net: 0VAC., PT6.
- new net: 100VAC., PT4.
- new net: PT14., V6., V7.
- new net: C17.2, RV7., SW2.
- new net: RV5., SW2.
- new net: 120VAC., PT8.
- new net: C6.2, RL1., RV2., V1B.
- new net: BRN., SW3.
- new net: J2. (In), T1. (SB)
- now unconnected: PT1., PT1., PT3., PT3., PT6., PT6., PT7., PT8., V6., V6.
Other:
- moved on the sheet: C15, R21

Commit message: Actual modifications version 2006
Parts:
- C36: value C_Polarized -> 100uF/400V
Connections:
- net GND: now also C3.2
- net at FCR.: now also B., C33.1, R49.1; no longer TRF4.
- net at 0VAC.: now also TR2.; no longer PT3.
- net at 60VAC.: now also TR2.; no longer PT11.
- net at PT2.: now also PT3., PT6. (x2)
- net at V7.: now also C29.1, R44.2, V6.
- net at PT5.: now also PT6. (x2)
- net at PT6.: no longer PT5. (x2)
- net at PT4.: now also PT1., PT7.
- net at ff.: now also BLUE.; no longer TR3.
- net at BLUE.: now also OT6.; no longer ff.
- net at PT7.: now also PT1.
- net at PT1.: no longer PT7.
- net at U?.: now also OUT1.; no longer TR3.
- net at OUT1.: now also PS1., V6.; no longer U?.
- net at 120VAC.: now also TR2.; no longer PT5.
- net at TR3.: now also d.; no longer d.
- net at a.: now also d.; no longer TR3.
- net at s.: now also d.; no longer TR3.
- net at d.: now also s.; no longer TR3.
- net at PT7.: now also 100VAC.
- net at 100VAC.: now also TR2.; no longer PT7.
- net at 5VAC.: now also PT13.
- net at PT13.: now also C35.1, HTFS., R50.1, V8.; no longer 5VAC.
- net at BLK.: now also SW3.; no longer PT1.
- net at SW3.: now also BLU.; no longer BLK.
- net at 0VAC.: now also TR2.; no longer PT6.
- net at 100VAC.: now also TR2.; no longer PT4.
- net at V6., V7.: now also PT15.; no longer PT14.
- net at PT1.: now also PT8.
- net at PT8.: no longer PT1.
- net at SW2.: now also RV7.; no longer RV5.
- net at RV7.: now also R23.2; no longer SW2.
- net at 120VAC.: now also TR2.; no longer PT8.
- net at PT2.: now also PT3.
- net at PT3.: no longer PT2.
- net at PT5.: now also PT1., PT8.
- net at 0VAC.: now also PT12.
- net at PT12.: now also F7.1; no longer 0VAC.
- net at s.: now also a.; no longer d.
- net at a.: now also J6., J7.; no longer s.
- net at BRN.: now also F9.2; no longer SW3.
- net at BLU.: now also AC-Input1.; no longer SW3.
- net at PT3.: now also PT2.
- net at PT2.: no longer PT3.
- net at C3.1: now also D6.1 (K), D7.1 (K), F., M1. (-), V1., V2., V3., V4., V5.
- new net: FCR., TRF4.
- new net: 0VAC., PT3.
- new net: 0VAC., TR2. (x2)
- new net: D4.2 (A), J4., RL3.
- new net: D3.2 (A), J4., RL1., RLY2.
- new net: J4., PB1.
- new net: 60VAC., PT11.
- new net: J3. (In), R29.1, RL3., V5A., V5B.
- new net: OUT2., PS2., V7.
- new net: TR3., ff.
- new net: TR3., U?.
- new net: B., PS5., PS6.
- new net: J5., J6., J7., J8., J9., d.
- new net: C4.2, RLY2., RV1.
- new net: 120VAC., PT5.
- new net: R19.2, RLY2., V2B.
- new net: RLY2., RV4.
- new net: TR3., d.
- new net: TR3., a.
- new net: TR3., s.
- new net: BLK., PT1.
- new net: 0VAC., PT6.
- new net: 100VAC., PT4.
- new net: PT14., V6., V7.
- new net: C17.2, RV7., SW2.
- new net: RV5., SW2.
- new net: 120VAC., PT8.
- new net: C6.2, RL1., RV2., V1B.
- new net: BRN., SW3.
- new net: J2. (In), T1. (SB)
- now unconnected: PT1., PT1., PT3., PT3., PT6., PT6., PT7., PT8., V6., V6.
Other:
- note added: "13V"
- note added: "279V"
- note added: "299V"
- note added: "331V"
- note added: "406V"
- moved on the sheet: C3
Changed lines of the file:
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@@
 	(wire
 		(pts
+			(xy 234.95 268.478) (xy 234.95 272.288)
+		)
+		(stroke
+			(width 0)
+			(type default)
+			(color 0 0 255 1)
+		)
+	)
+	(wire
+		(pts
 			(xy 73.914 119.634) (xy 68.834 119.634)
 		)
@@
 	(wire
 		(pts
-			(xy 251.206 243.84) (xy 251.46 243.84)
-		)
-		(stroke
-			(width 0)
-			(type default)
-			(color 0 0 255 1)
-		)
-	)
-	(wire
-		(pts
 			(xy 290.068 158.242) (xy 295.656 158.242)
 		)
@@
 	(wire
 		(pts
+			(xy 234.95 276.352) (xy 234.95 280.67)
+		)
+		(stroke
+			(width 0)
+			(type default)
+			(color 0 0 255 1)
+		)
+	)
+	(wire
+		(pts
 			(xy 173.736 36.068) (xy 177.8 36.068)
 		)
@@
 	(wire
 		(pts
-			(xy 234.95 277.114) (xy 234.95 280.67)
-		)
-		(stroke
-			(width 0)
-			(type default)
-			(color 0 0 255 1)
-		)
-	)
-	(wire
-		(pts
 			(xy 150.368 219.456) (xy 152.654 219.456)
 		)
@@
 	(wire
 		(pts
-			(xy 251.46 243.84) (xy 251.46 245.11)
+			(xy 251.206 243.84) (xy 251.206 245.11)
 		)
 		(stroke
@@
 		)
 	)
-	(wire
-		(pts
-			(xy 234.95 268.478) (xy 234.95 269.494)
-		)
-		(stroke
-			(width 0)
-			(type default)
-			(color 0 0 255 1)
-		)
-	)
 	(rectangle
 		(start 53.594 268.478)
@@
 		)
 	)
+	(text "279V"
+		(exclude_from_sim no)
+		(at 368.046 206.502 0)
+		(effects
+			(font
+				(size 1.27 1.27)
+				(thickness 0.254)
+				(bold yes)
+				(color 255 0 0 1)
+			)
+		)
+	)
 	(text "TREBLE"
 		(exclude_from_sim no)
@@
 		)
 	)
+	(text "299V"
+		(exclude_from_sim no)
+		(at 354.076 206.502 0)
+		(effects
+			(font
+				(size 1.27 1.27)
+				(thickness 0.254)
+				(bold yes)
+				(color 255 0 0 1)
+			)
+		)
+	)
 	(text "RED"
 		(exclude_from_sim no)
@@
 		)
 	)
+	(text "331V"
+		(exclude_from_sim no)
+		(at 339.598 206.502 0)
+		(effects
+			(font
+				(size 1.27 1.27)
+				(thickness 0.254)
+				(bold yes)
+				(color 255 0 0 1)
+			)
+		)
+	)
 	(text "BLK"
 		(exclude_from_sim no)
@@
 		)
 	)
+	(text "406V"
+		(exclude_from_sim no)
+		(at 325.628 206.502 0)
+		(effects
+			(font
+				(size 1.27 1.27)
+				(thickness 0.254)
+				(bold yes)
+				(color 255 0 0 1)
+			)
+		)
+	)
 	(text "@2AMP"
 		(exclude_from_sim no)
@@
 		)
 	)
+	(text "13V"
+		(exclude_from_sim no)
+		(at 279.908 259.334 0)
+		(effects
+			(font
+				(size 1.27 1.27)
+				(thickness 0.254)
+				(bold yes)
+				(color 255 0 0 1)
+			)
+		)
+	)
 	(text "RED"
 		(exclude_from_sim no)
@@
 		)
 	)
+	(text "406V"
+		(exclude_from_sim no)
+		(at 274.32 206.502 0)
+		(effects
+			(font
+				(size 1.27 1.27)
+				(thickness 0.254)
+				(bold yes)
+				(color 255 0 0 1)
+			)
+		)
+	)
 	(text "RED"
 		(exclude_from_sim no)
@@
 		(lib_name "C_Polarized_1")
 		(lib_id "Device:C_Polarized")
-		(at 234.95 273.304 0)
+		(at 234.95 274.32 0)
 		(unit 1)
 		(exclude_from_sim no)
@@
 		(dnp no)
 		(property "Reference" "C3"
-			(at 237.49 273.304 0)
+			(at 237.49 274.32 0)
 			(effects
 				(font
@@
 		)
 		(property "Value" "471/1KV"
-			(at 235.204 275.336 0)
+			(at 235.204 276.352 0)
 			(effects
 				(font
@@
 		)
 		(property "Footprint" ""
-			(at 235.9152 277.114 0)
+			(at 235.9152 278.13 0)
 			(effects
 				(font
@@
 		)
 		(property "Datasheet" "~"
-			(at 234.95 273.304 0)
+			(at 234.95 274.32 0)
 			(effects
 				(font
@@
 		)
 		(property "Description" "Unpolarized capacitor"
-			(at 234.95 273.304 0)
+			(at 234.95 274.32 0)
 			(effects
 				(font
@@
 		(dnp no)
 		(property "Reference" "C35"
-			(at 254.254 220.472 0)
+			(at 254 221.488 0)
 			(effects
 				(font
@@
 		)
 		(property "Value" "100uF/400V"
-			(at 254.508 222.504 0)
+			(at 254 223.012 0)
 			(effects
 				(font
@@
 		(dnp no)
 		(property "Reference" "C36"
-			(at 253.746 235.712 0)
+			(at 254 235.966 0)
 			(effects
 				(font
@@
 			)
 		)
-		(property "Value" "C_Polarized"
-			(at 255.27 237.363 0)
+		(property "Value" "100uF/400V"
+			(at 254 237.49 0)
 			(effects
 				(font
@@
 	(symbol
 		(lib_id "power:GND")
-		(at 251.46 245.11 0)
+		(at 251.206 245.11 0)
 		(unit 1)
 		(exclude_from_sim no)
@@
 		(fields_autoplaced yes)
 		(property "Reference" "#PWR03"
-			(at 251.46 251.46 0)
+			(at 251.206 251.46 0)
 			(effects
 				(font
@@
 		)
 		(property "Value" "GND"
-			(at 251.46 250.19 0)
+			(at 251.206 250.19 0)
 			(effects
 				(font
@@
 		)
 		(property "Footprint" ""
-			(at 251.46 245.11 0)
+			(at 251.206 245.11 0)
 			(effects
 				(font
@@
 		)
 		(property "Datasheet" ""
-			(at 251.46 245.11 0)
+			(at 251.206 245.11 0)
 			(effects
 				(font
@@
 		)
 		(property "Description" "Power symbol creates a global label with name \"GND\" , ground"
-			(at 251.46 245.11 0)
+			(at 251.206 245.11 0)
 			(effects
 				(font
