File: Schematics/Epiphone Blues Custom 30.kicad_sch (KiCad schematic)
At the start: 274 parts, among them J3 Conn_Coaxial_Power, M1 Fan, SW2 EQ mode, SW3 POWER, SW4 STANDBY, SW5 PENTODE

Commit message: Modified C3,C5,C6,C15,R15,R21
Parts:
- removed SW4: STANDBY, symbol Epi-BC-30:2PST
- added R15': 5K6/1W, symbol Device:R
- added R21': 2K2/1W, symbol Device:R
- added R52, R53: 68R/25W, symbol Device:R
- added SW-C3, SW-C5, SW-C6: ~, symbol Epi-BC-30:SPST-Small
- C15: value 22uF/35V -> 2.2uF/35V
- C3: value 22000uF/25V -> 101/1KV
Connections:
- net GND: now also R15'.1, R21'.1; no longer C3.2
- net at FCR.: now also B., C33.1, R49.1; no longer TRF4.
- net at C2.2, R5.1, R6.1: now also SW-C3., SW-C5.; no longer C3.1, C5.1
- net at SS1.: now also F4.1
- net at 0VAC.: now also TR2.; no longer PT3.
- net at 60VAC.: now also TR2.; no longer PT11.
- net at PT2.: now also PT3., PT6. (x2)
- net at V7.: now also C29.1, R44.2, V6.
- net at PT5.: now also PT6. (x2)
- net at PT6.: no longer PT5. (x2)
- net at C5.2, R6.2, RV2.: now also SW-C6.; no longer C6.1
- net at PT4.: now also PT1., PT7.
- net at ff.: now also BLUE.; no longer TR3.
- net at BLUE.: now also OT6.; no longer ff.
- net at PT7.: now also PT1.
- net at PT1.: no longer PT7.
- net at U?.: now also OUT1.; no longer TR3.
- net at OUT1.: now also PS1., V6.; no longer U?.
- net at 120VAC.: now also TR2.; no longer PT5.
- net at TR3.: now also d.; no longer d.
- net at a.: now also d.; no longer TR3.
- net at s.: now also d.; no longer TR3.
- net at d.: now also s.; no longer TR3.
- net at PT7.: now also 100VAC.
- net at 100VAC.: now also TR2.; no longer PT7.
- net at 5VAC.: now also PT13.
- net at PT13.: now also C35.1, HTFS., R50.1, V8.; no longer 5VAC.
- net at BLK.: now also SW3.; no longer PT1.
- net at SW3.: now also BLU.; no longer BLK.
- net at R15.1, V2A.: now also R15'.2
- net at 0VAC.: now also TR2.; no longer PT6.
- net at 100VAC.: now also TR2.; no longer PT4.
- net at V6., V7.: now also PT15.; no longer PT14.
- net at PT1.: now also PT8.
- net at PT8.: no longer PT1.
- net at SW2.: now also RV7.; no longer RV5.
- net at RV7.: now also R23.2; no longer SW2.
- net at 120VAC.: now also TR2.; no longer PT8.
- net at SS2.: now also R52.2
- net at 350VAC.: now also TR2. (x2)
- net at PT2.: now also PT3.
- net at PT3.: no longer PT2.
- net at PT5.: now also PT1., PT8.
- net at 0VAC.: now also PT12.
- net at PT12.: now also F7.1; no longer 0VAC.
- net at s.: now also a.; no longer d.
- net at a.: now also J6., J7.; no longer s.
- net at C15.1, R21.2, V2B.: now also R21'.2
- net at BRN.: now also F9.2; no longer SW3.
- net at BLU.: now also AC-Input1.; no longer SW3.
- net at PT3.: now also PT2.
- net at PT2.: no longer PT3.
- new net: D6.1 (K), D7.1 (K), F., M1. (-), V1., V2., V3., V4., V5.
- new net: FCR., TRF4.
- new net: R53.2, SS1.
- new net: 0VAC., PT3.
- new net: 0VAC., TR2. (x2)
- new net: D4.2 (A), J4., RL3.
- new net: D3.2 (A), J4., RL1., RLY2.
- new net: J4., PB1.
- new net: 60VAC., PT11.
- new net: J3. (In), R29.1, RL3., V5A., V5B.
- new net: OUT2., PS2., V7.
- new net: C5.1, SW-C5.
- new net: TR3., ff.
- new net: TR3., U?.
- new net: C3.1, SW-C3.
- new net: B., PS5., PS6.
- new net: J5., J6., J7., J8., J9., d.
- new net: C4.2, RLY2., RV1.
- new net: 120VAC., PT5.
- new net: R19.2, RLY2., V2B.
- new net: RLY2., RV4.
- new net: TR3., d.
- new net: TR3., a.
- new net: TR3., s.
- new net: BLK., PT1.
- new net: 0VAC., PT6.
- new net: 100VAC., PT4.
- new net: PT14., V6., V7.
- new net: C17.2, RV7., SW2.
- new net: RV5., SW2.
- new net: 120VAC., PT8.
- new net: C6.2, RL1., RV2., V1B.
- new net: BRN., SW3.
- new net: 350VAC., R53.1
- new net: J2. (In), T1. (SB)
- new net: C6.1, SW-C6.
- new net: 350VAC., R52.1
- now unconnected: C3.1, PT1., PT1., PT3., PT3., PT6., PT6., PT7., PT8., V6., V6.
Other:
- note removed: "TEST"
- moved on the sheet: C15, C3, C5, C6, R21

Commit message: Modified C3,C5,C6,C15,R15,R21
Parts:
- removed R39: 220K/1W, symbol Device:R
- added VR9: B1M, symbol Device:R_Potentiometer
Connections:
- net GND: now also VR9.
- net at FCR.: now also B., C33.1, R49.1; no longer TRF4.
- net at 0VAC.: now also TR2.; no longer PT3.
- net at 60VAC.: now also TR2.; no longer PT11.
- net at PT2.: now also PT3., PT6. (x2)
- net at V7.: now also C29.1, R44.2, V6.
- net at PT5.: now also PT6. (x2)
- net at PT6.: no longer PT5. (x2)
- net at PT4.: now also PT1., PT7.
- net at ff.: now also BLUE.; no longer TR3.
- net at BLUE.: now also OT6.; no longer ff.
- net at PT7.: now also PT1.
- net at PT1.: no longer PT7.
- net at U?.: now also OUT1.; no longer TR3.
- net at OUT1.: now also PS1., V6.; no longer U?.
- net at 120VAC.: now also TR2.; no longer PT5.
- net at TR3.: now also d.; no longer d.
- net at a.: now also d.; no longer TR3.
- net at s.: now also d.; no longer TR3.
- net at d.: now also s.; no longer TR3.
- net at PT7.: now also 100VAC.
- net at 100VAC.: now also TR2.; no longer PT7.
- net at 5VAC.: now also PT13.
- net at PT13.: now also C35.1, HTFS., R50.1, V8.; no longer 5VAC.
- net at BLK.: now also SW3.; no longer PT1.
- net at SW3.: now also BLU.; no longer BLK.
- net at C27.2, R31.2, R32.1: now also VR9.
- net at 0VAC.: now also TR2.; no longer PT6.
- net at 100VAC.: now also TR2.; no longer PT4.
- net at V6., V7.: now also PT15.; no longer PT14.
- net at PT1.: now also PT8.
- net at PT8.: no longer PT1.
- net at SW2.: now also RV7.; no longer RV5.
- net at RV7.: now also R23.2; no longer SW2.
- net at 120VAC.: now also TR2.; no longer PT8.
- net at PT2.: now also PT3.
- net at PT3.: no longer PT2.
- net at PT5.: now also PT1., PT8.
- net at 0VAC.: now also PT12.
- net at PT12.: now also F7.1; no longer 0VAC.
- net at s.: now also a.; no longer d.
- net at a.: now also J6., J7.; no longer s.
- net at BRN.: now also F9.2; no longer SW3.
- net at BLU.: now also AC-Input1.; no longer SW3.
- net at PT3.: now also PT2.
- net at PT2.: no longer PT3.
- new net: D6.1 (K), D7.1 (K), F., M1. (-), V1., V2., V3., V4., V5.
- new net: FCR., TRF4.
- new net: 0VAC., PT3.
- new net: 0VAC., TR2. (x2)
- new net: D4.2 (A), J4., RL3.
- new net: D3.2 (A), J4., RL1., RLY2.
- new net: J4., PB1.
- new net: 60VAC., PT11.
- new net: J3. (In), R29.1, RL3., V5A., V5B.
- new net: OUT2., PS2., V7.
- new net: TR3., ff.
- new net: TR3., U?.
- new net: B., PS5., PS6.
- new net: J5., J6., J7., J8., J9., d.
- new net: C4.2, RLY2., RV1.
- new net: 120VAC., PT5.
- new net: R19.2, RLY2., V2B.
- new net: RLY2., RV4.
- new net: TR3., d.
- new net: TR3., a.
- new net: TR3., s.
- new net: BLK., PT1.
- new net: 0VAC., PT6.
- new net: 100VAC., PT4.
- new net: PT14., V6., V7.
- new net: C17.2, RV7., SW2.
- new net: RV5., SW2.
- new net: 120VAC., PT8.
- new net: C6.2, RL1., RV2., V1B.
- new net: BRN., SW3.
- new net: J2. (In), T1. (SB)
- now unconnected: PT1., PT1., PT3., PT3., PT6., PT6., PT7., PT8., V6., V6.
Other:
- note added: "MASTER VOLUME"
Changed lines of the file:
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@@
 	)
 	(junction
+		(at 314.452 101.346)
+		(diameter 0)
+		(color 0 0 0 0)
+	)
+	(junction
 		(at 336.804 188.976)
 		(diameter 0)
@@
 		(color 194 0 0 1)
 	)
-	(junction
-		(at 314.452 101.346)
-		(diameter 0)
-		(color 194 0 0 1)
-	)
 	(wire
 		(pts
@@
 	(wire
 		(pts
+			(xy 307.34 101.346) (xy 314.452 101.346)
+		)
+		(stroke
+			(width 0)
+			(type default)
+		)
+	)
+	(wire
+		(pts
 			(xy 261.366 280.67) (xy 261.366 277.876)
 		)
@@
 	(wire
 		(pts
+			(xy 314.452 101.346) (xy 314.452 102.87)
+		)
+		(stroke
+			(width 0)
+			(type default)
+		)
+	)
+	(wire
+		(pts
 			(xy 212.598 254) (xy 212.598 252.476)
 		)
@@
 	(wire
 		(pts
-			(xy 311.15 101.346) (xy 314.452 101.346)
-		)
-		(stroke
-			(width 0)
-			(type default)
-			(color 0 0 255 1)
-		)
-	)
-	(wire
-		(pts
 			(xy 312.42 152.4) (xy 273.558 152.4)
 		)
@@
 	(wire
 		(pts
-			(xy 300.228 101.346) (xy 303.53 101.346)
+			(xy 300.228 105.156) (xy 303.53 105.156)
 		)
 		(stroke
@@
 	(wire
 		(pts
+			(xy 300.228 105.156) (xy 300.228 101.346)
+		)
+		(stroke
+			(width 0)
+			(type default)
+			(color 0 0 255 1)
+		)
+	)
+	(wire
+		(pts
 			(xy 72.898 246.126) (xy 72.898 251.714)
 		)
@@
 	(wire
 		(pts
-			(xy 314.452 102.87) (xy 314.452 101.346)
-		)
-		(stroke
-			(width 0)
-			(type default)
-			(color 0 0 255 1)
-		)
-	)
-	(wire
-		(pts
 			(xy 146.304 264.16) (xy 146.304 266.954)
 		)
@@
 		)
 	)
+	(text "MASTER VOLUME"
+		(exclude_from_sim no)
+		(at 307.34 109.728 0)
+		(effects
+			(font
+				(size 1.27 1.27)
+				(thickness 0.254)
+				(bold yes)
+				(color 0 132 0 1)
+			)
+		)
+	)
 	(text "240VAC"
 		(exclude_from_sim no)
@@
 	)
 	(symbol
-		(lib_name "Epi-BC-30:SPST-Small")
 		(lib_id "Epi-BC-30:SPST-Small")
 		(at 108.712 55.118 90)
@@
 	)
 	(symbol
-		(lib_name "Epi-BC-30:SPST-Small")
 		(lib_id "Epi-BC-30:SPST-Small")
 		(at 106.68 38.354 0)
@@
 	)
 	(symbol
+		(lib_name "R_Potentiometer_8")
+		(lib_id "Device:R_Potentiometer")
+		(at 307.34 105.156 90)
+		(unit 1)
+		(exclude_from_sim no)
+		(in_bom yes)
+		(on_board yes)
+		(dnp no)
+		(property "Reference" "VR9"
+			(at 307.34 107.442 90)
+			(effects
+				(font
+					(size 0.889 0.889)
+				)
+			)
+		)
+		(property "Value" "B1M"
+			(at 307.34 105.156 90)
+			(effects
+				(font
+					(size 0.889 0.889)
+					(color 0 0 0 1)
+				)
+			)
+		)
+		(property "Footprint" ""
+			(at 307.34 105.156 0)
+			(effects
+				(font
+					(size 1.27 1.27)
+				)
+				(hide yes)
+			)
+		)
+		(property "Datasheet" "~"
+			(at 307.34 105.156 0)
+			(effects
+				(font
+					(size 1.27 1.27)
+				)
+				(hide yes)
+			)
+		)
+		(property "Description" "Potentiometer"
+			(at 307.34 105.156 0)
+			(effects
+				(font
+					(size 1.27 1.27)
+				)
+				(hide yes)
+			)
+		)
+		(pin ""
+		)
+		(pin ""
+		)
+		(pin ""
+		)
+		(instances
+			(project ""
+				(path "/a50ba6b9-ea4a-46b2-bba0-285d6470a187"
+					(reference "VR9")
+					(unit 1)
+				)
+			)
+		)
+	)
+	(symbol
 		(lib_id "Epi-BC-30:Label")
 		(at 62.992 215.138 180)
@@
 	)
 	(symbol
-		(lib_name "Epi-BC-30:SPST-Small")
 		(lib_id "Epi-BC-30:SPST-Small")
 		(at 122.936 38.1 90)
@@
 					(unit 1)
 				)
-			)
-		)
-	)
-	(symbol
-		(lib_id "Device:R")
-		(at 307.34 101.346 270)
-		(unit 1)
-		(exclude_from_sim no)
-		(in_bom yes)
-		(on_board yes)
-		(dnp no)
-		(property "Reference" "R39"
-			(at 307.3564 101.3387 90)
-			(effects
-				(font
-					(size 0.889 0.889)
-				)
-			)
-		)
-		(property "Value" "220K/1W"
-			(at 307.6104 103.6247 90)
-			(effects
-				(font
-					(size 0.889 0.889)
-					(color 194 0 0 1)
-				)
-			)
-		)
-		(property "Footprint" ""
-			(at 307.34 99.568 90)
-			(effects
-				(font
-					(size 0.889 0.889)
-				)
-				(hide yes)
-			)
-		)
-		(property "Datasheet" "~"
-			(at 307.34 101.346 0)
-			(effects
-				(font
-					(size 0.889 0.889)
-				)
-				(hide yes)
-			)
-		)
-		(property "Description" "Resistor"
-			(at 307.34 101.346 0)
-			(effects
-				(font
-					(size 0.889 0.889)
-				)
-				(hide yes)
-			)
-		)
-		(pin "2"
-		)
-		(pin "1"
-		)
-		(instances
-			(project ""
-				(path "/a50ba6b9-ea4a-46b2-bba0-285d6470a187"
-					(reference "R39")
-					(unit 1)
-				)

Commit message: Added master volume and completed sheets data
Connections:
- net at FCR.: now also B., C33.1, R49.1; no longer TRF4.
- net at 0VAC.: now also TR2.; no longer PT3.
- net at 60VAC.: now also TR2.; no longer PT11.
- net at PT2.: now also PT3., PT6. (x2)
- net at V7.: now also C29.1, R44.2, V6.
- net at PT5.: now also PT6. (x2)
- net at PT6.: no longer PT5. (x2)
- net at PT4.: now also PT1., PT7.
- net at ff.: now also BLUE.; no longer TR3.
- net at BLUE.: now also OT6.; no longer ff.
- net at PT7.: now also PT1.
- net at PT1.: no longer PT7.
- net at U?.: now also OUT1.; no longer TR3.
- net at OUT1.: now also PS1., V6.; no longer U?.
- net at 120VAC.: now also TR2.; no longer PT5.
- net at TR3.: now also d.; no longer d.
- net at a.: now also d.; no longer TR3.
- net at s.: now also d.; no longer TR3.
- net at d.: now also s.; no longer TR3.
- net at PT7.: now also 100VAC.
- net at 100VAC.: now also TR2.; no longer PT7.
- net at 5VAC.: now also PT13.
- net at PT13.: now also C35.1, HTFS., R50.1, V8.; no longer 5VAC.
- net at BLK.: now also SW3.; no longer PT1.
- net at SW3.: now also BLU.; no longer BLK.
- net at 0VAC.: now also TR2.; no longer PT6.
- net at 100VAC.: now also TR2.; no longer PT4.
- net at V6., V7.: now also PT15.; no longer PT14.
- net at PT1.: now also PT8.
- net at PT8.: no longer PT1.
- net at SW2.: now also RV7.; no longer RV5.
- net at RV7.: now also R23.2; no longer SW2.
- net at 120VAC.: now also TR2.; no longer PT8.
- net at PT2.: now also PT3.
- net at PT3.: no longer PT2.
- net at PT5.: now also PT1., PT8.
- net at 0VAC.: now also PT12.
- net at PT12.: now also F7.1; no longer 0VAC.
- net at s.: now also a.; no longer d.
- net at a.: now also J6., J7.; no longer s.
- net at BRN.: now also F9.2; no longer SW3.
- net at BLU.: now also AC-Input1.; no longer SW3.
- net at PT3.: now also PT2.
- net at PT2.: no longer PT3.
- new net: D6.1 (K), D7.1 (K), F., M1. (-), V1., V2., V3., V4., V5.
- new net: FCR., TRF4.
- new net: 0VAC., PT3.
- new net: 0VAC., TR2. (x2)
- new net: D4.2 (A), J4., RL3.
- new net: D3.2 (A), J4., RL1., RLY2.
- new net: J4., PB1.
- new net: 60VAC., PT11.
- new net: J3. (In), R29.1, RL3., V5A., V5B.
- new net: OUT2., PS2., V7.
- new net: TR3., ff.
- new net: TR3., U?.
- new net: B., PS5., PS6.
- new net: J5., J6., J7., J8., J9., d.
- new net: C4.2, RLY2., RV1.
- new net: 120VAC., PT5.
- new net: R19.2, RLY2., V2B.
- new net: RLY2., RV4.
- new net: TR3., d.
- new net: TR3., a.
- new net: TR3., s.
- new net: BLK., PT1.
- new net: 0VAC., PT6.
- new net: 100VAC., PT4.
- new net: PT14., V6., V7.
- new net: C17.2, RV7., SW2.
- new net: RV5., SW2.
- new net: 120VAC., PT8.
- new net: C6.2, RL1., RV2., V1B.
- new net: BRN., SW3.
- new net: J2. (In), T1. (SB)
- now unconnected: PT1., PT1., PT3., PT3., PT6., PT6., PT7., PT8., V6., V6.
Other:
- title: Epiphone Blues Custom 30 -> Epiphone Blues Custom 30 Version 2005
Changed lines of the file:
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@@
 	(paper "A3")
 	(title_block
-		(title "Epiphone Blues Custom 30")
+		(title "Epiphone Blues Custom 30 Version 2005")
 		(date "2024/11/02")
 		(rev "1")
 		(comment 1 "Creator : Geert Peeters")
+		(comment 2 "Modifications : C3,C5,C6,C15,R15,R22,R39")
+		(comment 3 "Added choke resistors 68R/25W")
+		(comment 4 "Added Master Volume")
 	)
 	(junction

Commit message: Added text to schematic
Connections:
- net at FCR.: now also B., C33.1, R49.1; no longer TRF4.
- net at 0VAC.: now also TR2.; no longer PT3.
- net at 60VAC.: now also TR2.; no longer PT11.
- net at PT2.: now also PT3., PT6. (x2)
- net at V7.: now also C29.1, R44.2, V6.
- net at PT5.: now also PT6. (x2)
- net at PT6.: no longer PT5. (x2)
- net at PT4.: now also PT1., PT7.
- net at ff.: now also BLUE.; no longer TR3.
- net at BLUE.: now also OT6.; no longer ff.
- net at PT7.: now also PT1.
- net at PT1.: no longer PT7.
- net at U?.: now also OUT1.; no longer TR3.
- net at OUT1.: now also PS1., V6.; no longer U?.
- net at 120VAC.: now also TR2.; no longer PT5.
- net at TR3.: now also d.; no longer d.
- net at a.: now also d.; no longer TR3.
- net at s.: now also d.; no longer TR3.
- net at d.: now also s.; no longer TR3.
- net at PT7.: now also 100VAC.
- net at 100VAC.: now also TR2.; no longer PT7.
- net at 5VAC.: now also PT13.
- net at PT13.: now also C35.1, HTFS., R50.1, V8.; no longer 5VAC.
- net at BLK.: now also SW3.; no longer PT1.
- net at SW3.: now also BLU.; no longer BLK.
- net at 0VAC.: now also TR2.; no longer PT6.
- net at 100VAC.: now also TR2.; no longer PT4.
- net at V6., V7.: now also PT15.; no longer PT14.
- net at PT1.: now also PT8.
- net at PT8.: no longer PT1.
- net at SW2.: now also RV7.; no longer RV5.
- net at RV7.: now also R23.2; no longer SW2.
- net at 120VAC.: now also TR2.; no longer PT8.
- net at PT2.: now also PT3.
- net at PT3.: no longer PT2.
- net at PT5.: now also PT1., PT8.
- net at 0VAC.: now also PT12.
- net at PT12.: now also F7.1; no longer 0VAC.
- net at s.: now also a.; no longer d.
- net at a.: now also J6., J7.; no longer s.
- net at BRN.: now also F9.2; no longer SW3.
- net at BLU.: now also AC-Input1.; no longer SW3.
- net at PT3.: now also PT2.
- net at PT2.: no longer PT3.
- new net: D6.1 (K), D7.1 (K), F., M1. (-), V1., V2., V3., V4., V5.
- new net: FCR., TRF4.
- new net: 0VAC., PT3.
- new net: 0VAC., TR2. (x2)
- new net: D4.2 (A), J4., RL3.
- new net: D3.2 (A), J4., RL1., RLY2.
- new net: J4., PB1.
- new net: 60VAC., PT11.
- new net: J3. (In), R29.1, RL3., V5A., V5B.
- new net: OUT2., PS2., V7.
- new net: TR3., ff.
- new net: TR3., U?.
- new net: B., PS5., PS6.
- new net: J5., J6., J7., J8., J9., d.
- new net: C4.2, RLY2., RV1.
- new net: 120VAC., PT5.
- new net: R19.2, RLY2., V2B.
- new net: RLY2., RV4.
- new net: TR3., d.
- new net: TR3., a.
- new net: TR3., s.
- new net: BLK., PT1.
- new net: 0VAC., PT6.
- new net: 100VAC., PT4.
- new net: PT14., V6., V7.
- new net: C17.2, RV7., SW2.
- new net: RV5., SW2.
- new net: 120VAC., PT8.
- new net: C6.2, RL1., RV2., V1B.
- new net: BRN., SW3.
- new net: J2. (In), T1. (SB)
- now unconnected: PT1., PT1., PT3., PT3., PT6., PT6., PT7., PT8., V6., V6.
Other:
- note added: "TEST"
Changed lines of the file:
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@@
+		)
+	)
+	(text "TEST"
+		(exclude_from_sim no)
+		(at 36.83 140.97 0)
+		(effects
+			(font
+				(size 5.08 5.08)
+				(thickness 1.016)
+				(bold yes)
+				(color 255 0 0 1)
+			)
 		)
 	)

Commit message: changed color of master volume
Connections:
- net at FCR.: now also B., C33.1, R49.1; no longer TRF4.
- net at 0VAC.: now also TR2.; no longer PT3.
- net at 60VAC.: now also TR2.; no longer PT11.
- net at PT2.: now also PT3., PT6. (x2)
- net at V7.: now also C29.1, R44.2, V6.
- net at PT5.: now also PT6. (x2)
- net at PT6.: no longer PT5. (x2)
- net at PT4.: now also PT1., PT7.
- net at ff.: now also BLUE.; no longer TR3.
- net at BLUE.: now also OT6.; no longer ff.
- net at PT7.: now also PT1.
- net at PT1.: no longer PT7.
- net at U?.: now also OUT1.; no longer TR3.
- net at OUT1.: now also PS1., V6.; no longer U?.
- net at 120VAC.: now also TR2.; no longer PT5.
- net at TR3.: now also d.; no longer d.
- net at a.: now also d.; no longer TR3.
- net at s.: now also d.; no longer TR3.
- net at d.: now also s.; no longer TR3.
- net at PT7.: now also 100VAC.
- net at 100VAC.: now also TR2.; no longer PT7.
- net at 5VAC.: now also PT13.
- net at PT13.: now also C35.1, HTFS., R50.1, V8.; no longer 5VAC.
- net at BLK.: now also SW3.; no longer PT1.
- net at SW3.: now also BLU.; no longer BLK.
- net at 0VAC.: now also TR2.; no longer PT6.
- net at 100VAC.: now also TR2.; no longer PT4.
- net at V6., V7.: now also PT15.; no longer PT14.
- net at PT1.: now also PT8.
- net at PT8.: no longer PT1.
- net at SW2.: now also RV7.; no longer RV5.
- net at RV7.: now also R23.2; no longer SW2.
- net at 120VAC.: now also TR2.; no longer PT8.
- net at PT2.: now also PT3.
- net at PT3.: no longer PT2.
- net at PT5.: now also PT1., PT8.
- net at 0VAC.: now also PT12.
- net at PT12.: now also F7.1; no longer 0VAC.
- net at s.: now also a.; no longer d.
- net at a.: now also J6., J7.; no longer s.
- net at BRN.: now also F9.2; no longer SW3.
- net at BLU.: now also AC-Input1.; no longer SW3.
- net at PT3.: now also PT2.
- net at PT2.: no longer PT3.
- new net: D6.1 (K), D7.1 (K), F., M1. (-), V1., V2., V3., V4., V5.
- new net: FCR., TRF4.
- new net: 0VAC., PT3.
- new net: 0VAC., TR2. (x2)
- new net: D4.2 (A), J4., RL3.
- new net: D3.2 (A), J4., RL1., RLY2.
- new net: J4., PB1.
- new net: 60VAC., PT11.
- new net: J3. (In), R29.1, RL3., V5A., V5B.
- new net: OUT2., PS2., V7.
- new net: TR3., ff.
- new net: TR3., U?.
- new net: B., PS5., PS6.
- new net: J5., J6., J7., J8., J9., d.
- new net: C4.2, RLY2., RV1.
- new net: 120VAC., PT5.
- new net: R19.2, RLY2., V2B.
- new net: RLY2., RV4.
- new net: TR3., d.
- new net: TR3., a.
- new net: TR3., s.
- new net: BLK., PT1.
- new net: 0VAC., PT6.
- new net: 100VAC., PT4.
- new net: PT14., V6., V7.
- new net: C17.2, RV7., SW2.
- new net: RV5., SW2.
- new net: 120VAC., PT8.
- new net: C6.2, RL1., RV2., V1B.
- new net: BRN., SW3.
- new net: J2. (In), T1. (SB)
- now unconnected: PT1., PT1., PT3., PT3., PT6., PT6., PT7., PT8., V6., V6.
Other:
- note removed: "TEST"
Changed lines of the file:
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@@
-		)
-	)
-	(text "TEST"
-		(exclude_from_sim no)
-		(at 36.83 140.97 0)
-		(effects
-			(font
-				(size 5.08 5.08)
-				(thickness 1.016)
-				(bold yes)
-				(color 255 0 0 1)
-			)
 		)
 	)
