File: schematics/epiphone-blues-custom-30.kicad_sch (KiCad schematic)
At the start: 288 parts, among them J10 Midi In, J3 Conn_Coaxial_Power, M1 Fan, M2 Servo, SW2 EQ mode, SW3 POWER, SW5 PENTODE, U1 6N138

Commit message: Bestanden weer juiste extentie gegeven
Parts:
- removed SW-C3, SW-C5, SW-C6: (no value), symbol Epi-BC-30:SPST-Small
- added R6': 820K/1W, symbol Device:R
Connections:
- net Earth: no longer 0VAC., 0VAC., AC-Input1., TR2.
- net GND: no longer J1., M1. (-), RL1., V1., V2., V3., V4., V5.
- net at FCR.: now also B., C33.1, R49.1; no longer TRF4.
- net at C2.2, R5.1, R6.1: now also C3.1, C5.1, R6'.2
- net at R43.1: no longer V7.
- net at TR2.: now also 350VAC.; no longer 0VAC.
- net at 60VAC.: no longer PT11.
- net at PT2.: now also PT3., PT6. (x2)
- net at V7.: now also R46.2
- net at C29.1, R44.2: no longer V6., V7.
- net at PT5.: now also PT6. (x2)
- net at PT6.: no longer PT5. (x2)
- net at C5.2, R6.2, RV2.: now also C6.1, R6'.1
- net at PT4.: now also PT1., PT7.
- net at PS2.: now also OUT2.; no longer SW5.
- net at BLUE.: no longer ff.
- net at PT7.: now also PT1.
- net at PT1.: no longer PT7.
- net at U?.: now also OUT1.; no longer TR3.
- net at OUT1.: now also PS1.; no longer U?.
- net at D3.1 (K), D4.1 (K), F.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: no longer RLY2.
- net at 120VAC.: now also TR2.; no longer PT5.
- net at R19.2, V2B.: no longer RLY2.
- net at TR3.: now also s.; no longer d.
- net at a.: no longer TR3. (x2)
- net at s.: no longer TR3.
- net at d.: no longer TR3.
- net at PS4.: no longer SW5.
- net at PT7.: now also 100VAC.
- net at 100VAC.: no longer PT7.
- net at 11.5VAC.: no longer PT10.
- net at PT13.: no longer 5VAC.
- net at SW3.: now also BRN.; no longer BLK.
- net at d.: no longer a.
- net at C19.2: no longer SW2.
- net at F6.1: no longer 3.15VAC.
- net at PT1.: now also PT8.
- net at PT8.: no longer PT1.
- net at SW2.: now also RV7.; no longer RV5.
- net at R24.2: no longer SW2.
- net at RV7.: now also R23.2; no longer SW2.
- net at 120VAC.: now also TR2.; no longer PT8.
- net at PT2.: now also PT3.
- net at PT3.: no longer PT2.
- net at R12.1: no longer RL1.
- net at PT9.: no longer 0VAC.
- net at PT5.: now also PT1., PT8.
- net at 0VAC.: now also PT12.
- net at PT12.: now also F7.1; no longer 0VAC.
- net at d.: no longer s.
- net at s.: now also a.; no longer d.
- net at a.: now also J6., J7.; no longer s.
- net at BRN.: now also F9.2; no longer SW3.
- net at BLU.: no longer SW3.
- net at R53.1: no longer 350VAC.
- net at F5.1: no longer 3.15VAC.
- net at PT3.: now also PT2.
- net at PT2.: no longer PT3.
- net at R42.2: no longer V6.
- net at SW5.: now also PS1.; no longer PS3.
- net at PS6.: no longer SW5.
- net at 350VAC.: no longer TR2. (x2)
- net at 0VAC.: no longer TR2. (x2)
- net at AC-Input1.: no longer BLU.
- net at F7.2: no longer V8.
- net at R52.1: no longer 350VAC.
- net at 3.15VAC.: no longer TR2.
- new net: D6.1 (K), D7.1 (K), F., M1. (-)
- new net: D3.2 (A), J4., RLY2.
- new net: R29.1, RL3., V5A., V5B.
- new net: TR3., U?.
- new net: B., PS5., PS6.
- new net: J8., d.
- new net: C4.2, RV1.
- new net: 120VAC., PT5.
- new net: J9., f.
- new net: PT15., V7.
- new net: C35.1, PT13., R50.1, V8.
- new net: C17.2, RV7., SW2.
- new net: 120VAC., PT8.
- new net: RV2., V1B.
- new net: PT14., V6.
- new net: J2. (Ext), T1. (SA)
- new net: 0VAC., TR2.
- now unconnected: 100VAC., 11.5VAC., 60VAC., C6.2, D4.2 (A), HTFS., J6., J6., J9., J9., M1. (-), PS6., PT1., PT1., PT13., PT3., PT3., PT6., PT6., PT7., PT8., V1., V2., V3., V4., V5., V6., V6., V6.
Other:
- moved on the sheet: 0VAC, 100VAC, 120VAC, 3.15VAC, 350VAC, 60VAC, B, BLK, BLUE, BRN, C, C11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
