File: schematics/phase-inverter.kicad_sch (KiCad schematic)
At the start: 286 parts, among them J10 Midi In, J3 Conn_Coaxial_Power, M1 Fan, M2 Servo, SW2 EQ mode, SW3 POWER, SW5 PENTODE, U1 6N138

Commit message: added partial schematics
Parts:
- removed OT5: OT6, symbol Epi-BC-30:Label
- removed RL2: (no value), symbol Epi-BC-30:Relays
- added RLY2: (no value), symbol Epi-BC-30:Relays
- added a: OT5, symbol Epi-BC-30:Label
- BLUE: value OT6 -> (none)
Connections:
- net GND: now also J2. (Ext), J3. (In), RV1., RV2., RV3., RV4., RV6., RV8., T1. (SA), VR9., RLY2.; no longer J2.2 (Ext), J3.2 (Ext), RL1., RV1.3, RV2.3, RV3.3, RV4.3, RV6.3, RV8.3, VR9.2
- net at D6.1 (K), D7.1 (K), F.: now also M1. (-)
- net at FCR.: now also B., C33.1, R49.1
- net at C2.2, R5.1, R6'.2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: now also C3.1, C5.1
- net at C3.2, C4.1, R5.2: now also RV1.; no longer RV1.1
- net at 0VAC.: now also PT3.
- net at PT3.: now also PT2.; no longer 0VAC.
- net at 0VAC.: now also TR2.
- net at TR2.: now also 350VAC.; no longer 0VAC.
- net at TRF4.: now also FCS.
- net at FCS.: now also OTCT.; no longer TRF4.
- net at PT2.: now also PT3., PT6. (x2)
- net at V5A., V5B.: now also C22.1, R30.2; no longer R29.1, RL3.
- net at J1.: now also R1.1, R2.1
- net at V7.: now also R46.2
- net at PT5.: now also PT6. (x2)
- net at PT6.: no longer PT5. (x2)
- net at C5.2: now also C6.1, R6'.1, R6.2, RV2.
- net at PT4.: now also PT1., PT7.
- net at PS2.: now also OUT2.
- net at OUT2.: now also a.; no longer PS2.
- net at ff.: now also TR3.; no longer BLUE.
- net at TR3.: now also s.; no longer ff.
- net at PT7.: now also PT1.
- net at PT1.: no longer PT7.
- net at U?.: now also OUT1.; no longer TR3.
- net at OUT1.: now also PS1.; no longer U?.
- net at V3A., V3B.: now also T1. (SA)
- net at a.: no longer OUT2.
- net at J8.: now also d.
- net at d.: now also d.; no longer J8.
- net at C4.2: now also RV1.; no longer RV1.2
- net at C23.2: now also RV8.; no longer RV8.1
- net at R31.1: now also RV8.; no longer RV8.2
- net at 120VAC.: now also TR2.; no longer PT5.
- net at C16.2: now also RV5.; no longer RV5.1
- net at d.: no longer d.
- net at PT2.: now also WHT.; no longer PT3.
- net at s.: no longer TR3.
- net at PT7.: now also 100VAC.
- net at 100VAC.: no longer PT7.
- net at PT10.: now also F1.1
- net at f.: now also d.; no longer J9.
- net at d.: no longer f.
- net at BLK.: now also PT1.
- net at PT1.: no longer BLK.
- net at C27.2, R31.2, R32.1: now also VR9.; no longer VR9.1
- net at d.: now also A.
- net at C19.2: no longer SW2.
- net at 0VAC.: now also PT6.
- net at PT6.: no longer 0VAC.
- net at 100VAC.: now also PT4.
- net at PT4.: no longer 100VAC.
- net at V7.: now also PT15.
- net at PT15.: now also F5.2; no longer V7.
- net at PT1.: now also PT8.
- net at PT8.: no longer PT1.
- net at SW2.: now also RV7.; no longer RV5.3
- net at R24.2: no longer SW2.
- net at s.: now also a.
- net at J6., J7.: now also a.
- net at R24.1, R25.1, R32.2: now also RV5.; no longer RV5.2
- net at 120VAC.: now also TR2.; no longer PT8.
- net at PT2.: now also PT3.
- net at PT3.: no longer PT2.
- net at OTCT.: now also HTFR.; no longer FCS.
- net at RL1.: now also R13.1
- net at R12.1: no longer RL1.
- net at PS1.: now also SW5.; no longer OUT1.
- net at PT5.: now also PT1., PT8.
- net at V1B.: now also C7.2, C9.1, R7.1; no longer RV2.2
- net at 0VAC.: now also PT12.
- net at PT12.: now also F7.1; no longer 0VAC.
- net at SW3.: now also BRN.
- net at BRN.: now also F9.2; no longer SW3.
- net at R18.1: now also RV4.; no longer RV4.1
- net at PT3.: now also PT2.
- net at PT2.: no longer PT3.
- net at C.: now also T1. (SA)
- net at 3.15VAC.: now also TR2.
- net at V8.: now also F4.2
- net at J5.: now also OT6.
- net at R23.2: now also RV7.; no longer RV7.3
- net at 0VAC.: no longer TR2.
- net at 350VAC.: no longer TR2.
- new net: D3.2 (A), J4., RLY2.
- new net: R29.1, RL3., V5A., V5B.
- new net: TR3., U?.
- new net: B., PS5., PS6.
- new net: 120VAC., PT5.
- new net: J9., f.
- new net: C18.1, RV6.
- new net: C17.2, RV7., SW2.
- new net: 120VAC., PT8.
- new net: RV2., V1B.
- new net: J2. (Ext), T1. (SA)
- new net: C14.2, RV3.
- new net: 0VAC., TR2.
- now unconnected: PS6., PT1., PT1., PT3., PT3., PT6., PT6., PT7., PT8.
Other:
- moved on the sheet: C3, C6, SW2
